Commit message: add new model with rotating propeller

File: f450/ros2_ws/src/f450_description/urdf/f450.urdf.xacro (robot description, xacro)
@@ -37,4 +37,46 @@
   </material>
   <!-- ========================= -->
+  <!-- Physical propeller macro -->
+  <!-- ========================= -->
+  <xacro:macro name="physical_propeller" params="idx x y yaw mat">
+    <link name="propeller_${idx}_link">
+      <!-- Cánh số 1 -->
+      <visual>
+        <origin xyz="0 0 0" rpy="0 0 ${yaw}"/>
+        <geometry>
+          <box size="${prop_length} ${prop_width} ${prop_height}"/>
+        </geometry>
+        <material name="${mat}"/>
+      </visual>
+      <!-- Cánh số 2, vuông góc với cánh số 1 -->
+      <visual>
+        <origin xyz="0 0 0" rpy="0 0 ${yaw + 1.57079632679}"/>
+        <geometry>
+          <box size="${prop_length} ${prop_width} ${prop_height}"/>
+        </geometry>
+        <material name="${mat}"/>
+      </visual>
+      <!-- Inertia nhỏ cho propeller -->
+      <inertial>
+        <origin xyz="0 0 0" rpy="0 0 0"/>
+        <mass value="0.012"/>
+        <inertia
+          ixx="0.000001"
+          ixy="0.0"
+          ixz="0.0"
+          iyy="0.000032"
+          iyz="0.0"
+          izz="0.000032"/>
+      </inertial>
+    </link>
+    <joint name="propeller_${idx}_joint" type="continuous">
+      <parent link="base_link"/>
+      <child link="propeller_${idx}_link"/>
+      <origin xyz="${x} ${y} 0.065" rpy="0 0 0"/>
+      <axis xyz="0 0 1"/>
+      <dynamics damping="0.0001" friction="0.0"/>
+    </joint>
+  </xacro:macro>
+  <!-- ========================= -->
   <!-- Base link: toàn bộ thân drone là 1 rigid body -->
   <!-- ========================= -->
@@ -114,33 +156,88 @@
       <material name="gray"/>
     </visual>
-    <!-- Propeller đơn giản -->
-    <visual>
-      <origin xyz="${arm_xy} ${arm_xy} 0.04" rpy="0 0 0.785398"/>
-      <geometry>
-        <box size="${prop_length} ${prop_width} ${prop_height}"/>
-      </geometry>
-      <material name="red"/>
-    </visual>
-    <visual>
-      <origin xyz="${arm_xy} -${arm_xy} 0.04" rpy="0 0 -0.785398"/>
-      <geometry>
-        <box size="${prop_length} ${prop_width} ${prop_height}"/>
-      </geometry>
-      <material name="white"/>
-    </visual>
-    <visual>
-      <origin xyz="-${arm_xy} -${arm_xy} 0.04" rpy="0 0 0.785398"/>
-      <geometry>
-        <box size="${prop_length} ${prop_width} ${prop_height}"/>
-      </geometry>
-      <material name="red"/>
-    </visual>
-    <visual>
-      <origin xyz="-${arm_xy} ${arm_xy} 0.04" rpy="0 0 -0.785398"/>
-      <geometry>
-        <box size="${prop_length} ${prop_width} ${prop_height}"/>
-      </geometry>
-      <material name="white"/>
-    </visual>
+    <!-- ========================= -->
+    <!-- Landing gear / càng đáp -->
+    <!-- ========================= -->
+    <!-- Skid trái -->
+    <visual>
+      <origin xyz="0 0.12 -0.17" rpy="0 0 0"/>
+      <geometry>
+        <box size="0.38 0.025 0.025"/>
+      </geometry>
+      <material name="gray"/>
+    </visual>
+    <collision>
+      <origin xyz="0 0.12 -0.17" rpy="0 0 0"/>
+      <geometry>
+        <box size="0.38 0.025 0.025"/>
+      </geometry>
+    </collision>
+    <!-- Skid phải -->
+    <visual>
+      <origin xyz="0 -0.12 -0.17" rpy="0 0 0"/>
+      <geometry>
+        <box size="0.38 0.025 0.025"/>
+      </geometry>
+      <material name="gray"/>
+    </visual>
+    <collision>
+      <origin xyz="0 -0.12 -0.17" rpy="0 0 0"/>
+      <geometry>
+        <box size="0.38 0.025 0.025"/>
+      </geometry>
+    </collision>
+    <!-- 4 thanh chống càng đáp -->
+    <visual>
+      <origin xyz="0.12 0.12 -0.095" rpy="0 0 0"/>
+      <geometry>
+        <box size="0.018 0.018 0.15"/>
+      </geometry>
+      <material name="gray"/>
+    </visual>
+    <collision>
+      <origin xyz="0.12 0.12 -0.095" rpy="0 0 0"/>
+      <geometry>
+        <box size="0.018 0.018 0.15"/>
+      </geometry>
+    </collision>
+    <visual>
+      <origin xyz="-0.12 0.12 -0.095" rpy="0 0 0"/>
+      <geometry>
+        <box size="0.018 0.018 0.15"/>
+      </geometry>
+      <material name="gray"/>
+    </visual>
+    <collision>
+      <origin xyz="-0.12 0.12 -0.095" rpy="0 0 0"/>
+      <geometry>
+        <box size="0.018 0.018 0.15"/>
+      </geometry>
+    </collision>
+    <visual>
+      <origin xyz="0.12 -0.12 -0.095" rpy="0 0 0"/>
+      <geometry>
+        <box size="0.018 0.018 0.15"/>
+      </geometry>
+      <material name="gray"/>
+    </visual>
+    <collision>
+      <origin xyz="0.12 -0.12 -0.095" rpy="0 0 0"/>
+      <geometry>
+        <box size="0.018 0.018 0.15"/>
+      </geometry>
+    </collision>
+    <visual>
+      <origin xyz="-0.12 -0.12 -0.095" rpy="0 0 0"/>
+      <geometry>
+        <box size="0.018 0.018 0.15"/>
+      </geometry>
+      <material name="gray"/>
+    </visual>
+    <collision>
+      <origin xyz="-0.12 -0.12 -0.095" rpy="0 0 0"/>
+      <geometry>
+        <box size="0.018 0.018 0.15"/>
+      </geometry>
+    </collision>
     <!-- Inertial của toàn bộ drone -->
     <inertial>
@@ -196,3 +293,30 @@
     <origin xyz="0.08 0 -0.03" rpy="0 0 0"/>
   </joint>
+  <!-- ========================= -->
+  <!-- 4 physical propellers -->
+  <!-- ========================= -->
+  <xacro:physical_propeller
+    idx="1"
+    x="${arm_xy}"
+    y="${arm_xy}"
+    yaw="0.785398"
+    mat="red"/>
+  <xacro:physical_propeller
+    idx="2"
+    x="${arm_xy}"
+    y="-${arm_xy}"
+    yaw="-0.785398"
+    mat="white"/>
+  <xacro:physical_propeller
+    idx="3"
+    x="-${arm_xy}"
+    y="-${arm_xy}"
+    yaw="0.785398"
+    mat="red"/>
+  <xacro:physical_propeller
+    idx="4"
+    x="-${arm_xy}"
+    y="${arm_xy}"
+    yaw="-0.785398"
+    mat="white"/>
 </robot>

Commit message: repair position of propeller

File: f450/ros2_ws/src/f450_description/urdf/f450.urdf.xacro (robot description, xacro)
@@ -18,7 +18,10 @@
   <xacro:property name="motor_radius" value="0.025"/>
   <xacro:property name="motor_height" value="0.025"/>
+  <xacro:property name="motor_frame_z" value="0.04"/>
   <xacro:property name="prop_length" value="0.18"/>
   <xacro:property name="prop_width" value="0.025"/>
   <xacro:property name="prop_height" value="0.004"/>
+  <xacro:property name="propeller_z" value="0.035"/>
+  <xacro:property name="propeller_motor_offset_z" value="${propeller_z - motor_frame_z}"/>
   <!-- ========================= -->
   <!-- Materials -->
@@ -39,17 +42,9 @@
   <!-- Physical propeller macro -->
   <!-- ========================= -->
-  <xacro:macro name="physical_propeller" params="idx x y yaw mat">
+  <xacro:macro name="physical_propeller" params="idx yaw mat">
     <link name="propeller_${idx}_link">
-      <!-- Cánh số 1 -->
+      <!-- Một cánh quạt -->
       <visual>
         <origin xyz="0 0 0" rpy="0 0 ${yaw}"/>
-        <geometry>
-          <box size="${prop_length} ${prop_width} ${prop_height}"/>
-        </geometry>
-        <material name="${mat}"/>
-      </visual>
-      <!-- Cánh số 2, vuông góc với cánh số 1 -->
-      <visual>
-        <origin xyz="0 0 0" rpy="0 0 ${yaw + 1.57079632679}"/>
         <geometry>
           <box size="${prop_length} ${prop_width} ${prop_height}"/>
@@ -71,7 +66,7 @@
     </link>
     <joint name="propeller_${idx}_joint" type="continuous">
-      <parent link="base_link"/>
+      <parent link="motor_${idx}_link"/>
       <child link="propeller_${idx}_link"/>
-      <origin xyz="${x} ${y} 0.065" rpy="0 0 0"/>
+      <origin xyz="0 0 ${propeller_motor_offset_z}" rpy="0 0 0"/>
       <axis xyz="0 0 1"/>
       <dynamics damping="0.0001" friction="0.0"/>
@@ -261,20 +256,20 @@
     <parent link="base_link"/>
     <child link="motor_1_link"/>
-    <origin xyz="${arm_xy} ${arm_xy} 0.04" rpy="0 0 0"/>
+    <origin xyz="${arm_xy} ${arm_xy} ${motor_frame_z}" rpy="0 0 0"/>
   </joint>
   <joint name="motor_2_joint" type="fixed">
     <parent link="base_link"/>
     <child link="motor_2_link"/>
-    <origin xyz="${arm_xy} -${arm_xy} 0.04" rpy="0 0 0"/>
+    <origin xyz="${arm_xy} -${arm_xy} ${motor_frame_z}" rpy="0 0 0"/>
   </joint>
   <joint name="motor_3_joint" type="fixed">
     <parent link="base_link"/>
     <child link="motor_3_link"/>
-    <origin xyz="-${arm_xy} -${arm_xy} 0.04" rpy="0 0 0"/>
+    <origin xyz="-${arm_xy} -${arm_xy} ${motor_frame_z}" rpy="0 0 0"/>
   </joint>
   <joint name="motor_4_joint" type="fixed">
     <parent link="base_link"/>
     <child link="motor_4_link"/>
-    <origin xyz="-${arm_xy} ${arm_xy} 0.04" rpy="0 0 0"/>
+    <origin xyz="-${arm_xy} ${arm_xy} ${motor_frame_z}" rpy="0 0 0"/>
   </joint>
   <!-- ========================= -->
@@ -298,24 +293,16 @@
   <xacro:physical_propeller
     idx="1"
-    x="${arm_xy}"
-    y="${arm_xy}"
     yaw="0.785398"
     mat="red"/>
   <xacro:physical_propeller
     idx="2"
-    x="${arm_xy}"
-    y="-${arm_xy}"
     yaw="-0.785398"
     mat="white"/>
   <xacro:physical_propeller
     idx="3"
-    x="-${arm_xy}"
-    y="-${arm_xy}"
     yaw="0.785398"
     mat="red"/>
   <xacro:physical_propeller
     idx="4"
-    x="-${arm_xy}"
-    y="${arm_xy}"
     yaw="-0.785398"
     mat="white"/>
